Commit message: Phase

File: src/smart_wheelchair_description/urdf/wheelchair.urdf (robot description, URDF)
Before this commit: robot smart_wheelchair, 5 links, 4 joints
Links:
- added link front_caster, mass 0.1; collision sphere radius=0.05; visual sphere radius=0.05
- added link rear_caster, mass 0.1; collision sphere radius=0.05; visual sphere radius=0.05
- link base_link: mass None -> 10.0; geometry collision box size=0.6 0.4 0.2; visual box size=0.6 0.4 0.2
- link camera_link: mass None -> 0.05; geometry collision box size=0.02 0.1 0.02; visual box size=0.02 0.1 0.02
- link left_wheel: mass None -> 1.0; geometry collision cylinder length=0.05 radius=0.1; visual cylinder length=0.05 radius=0.1
- link lidar_link: mass None -> 0.1; geometry collision cylinder length=0.05 radius=0.05; visual cylinder length=0.05 radius=0.05
- link right_wheel: mass None -> 1.0; geometry collision cylinder length=0.05 radius=0.1; visual cylinder length=0.05 radius=0.1
Joints:
- added joint front_caster_joint: type fixed, parent base_link, child front_caster, origin xyz=0.25 0 -0.1 rpy=0 0 0
- added joint rear_caster_joint: type fixed, parent base_link, child rear_caster, origin xyz=-0.25 0 -0.1 rpy=0 0 0

Commit message: finish demo

File: src/smart_wheelchair_description/urdf/wheelchair.urdf (robot description, URDF)
Before this commit: robot smart_wheelchair, 7 links, 6 joints
Joints:
- joint camera_joint: origin xyz=0.3 0 0.05 rpy=0 0 0 -> xyz=0.35 0 0.65 rpy=0 0 0
